File: payload/Payload_V01/Laser.sch (KiCad schematic (older format))
At the start: 0 parts

Commit message: added laser and photodiode schematics
Parts:
- added LD?: DJ532-40, symbol Payload_V01:DJ532-40
- added R?: 1k, symbol Device:R_US
- added RV?: 10k, symbol Device:R_POT_US
- added U?: MLD203CLN, symbol Payload_V01:MLD203CLN
Connections:
- new net: RV?.1, U?.5 (VREFOUT)
- new net: RV?.2, U?.6 (ISET/IMOD)
- new net: RV?.3, U?.4 (GND2)
- new net: LD?.2 (A), U?.14 (LDA)
- new net: LD?.3 (K), U?.11 (LDC)
- new net: R?.2, U?.12 (ISENS+)
- new net +5V: U?.1 (VIN1), U?.2 (VIN2)
- new net GND: U?.3 (GND1)
- new net LD_CURR: R?.1, U?.13 (ISENS-)
Changed lines of the file:
@@
 $Descr A4 11693 8268
 encoding utf-8
-Sheet 1 4
+Sheet 3 5
 Title ""
 Date ""
@@
 Comment4 ""
 $EndDescr
+$Comp
+L power:GND #PWR?
+U 1 1 5F18C650
+P 4450 3550
+F 0 "#PWR?" H 4450 3300 50  0001 C CNN
+F 1 "GND" H 4455 3377 50  0000 C CNN
+F 2 "" H 4450 3550 50  0001 C CNN
+F 3 "" H 4450 3550 50  0001 C CNN
+	1    4450 3550
+	1    0    0    -1
+$EndComp
+$Comp
+L power:+5V #PWR?
+U 1 1 5F18CD3D
+P 4900 3250
+F 0 "#PWR?" H 4900 3100 50  0001 C CNN
+F 1 "+5V" H 4915 3423 50  0000 C CNN
+F 2 "" H 4900 3250 50  0001 C CNN
+F 3 "" H 4900 3250 50  0001 C CNN
+	1    4900 3250
+	1    0    0    -1
+$EndComp
+Wire Wire Line
+	4900 3250 5150 3250
+Wire Wire Line
+	5150 3250 5150 3400
+Wire Wire Line
+	5150 3400 5300 3400
+Connection ~ 5150 3250
+Wire Wire Line
+	5150 3250 5300 3250
+$Comp
+L Device:R_POT_US RV?
+U 1 1 5F18DE7D
+P 5000 3850
+F 0 "RV?" V 4795 3850 50  0000 C CNN
+F 1 "10k" V 4886 3850 50  0000 C CNN
+F 2 "" H 5000 3850 50  0001 C CNN
+F 3 "~" H 5000 3850 50  0001 C CNN
+	1    5000 3850
+	0    1    1    0
+$EndComp
+Wire Wire Line
+	4450 3550 5300 3550
+Wire Wire Line
+	5150 3850 5300 3850
+Wire Wire Line
+	5300 3700 4850 3700
+Wire Wire Line
+	4850 3700 4850 3850
+Wire Wire Line
+	5300 4000 5000 4000
+$Comp
+L Payload_V01:DJ532-40 LD?
+U 1 1 5F1DD2C7
+P 6950 4000
+F 0 "LD?" V 6854 4147 50  0000 L CNN
+F 1 "DJ532-40" V 6945 4147 50  0000 L CNN
+F 2 "" H 6950 4000 50  0001 C CNN
+F 3 "" H 6950 4000 50  0001 C CNN
+	1    6950 4000
+	0    1    1    0
+$EndComp
+$Comp
+L Payload_V01:MLD203CLN U?
+U 1 1 5F1DFA85
+P 5850 3700
+F 0 "U?" H 5850 4415 50  0000 C CNN
+F 1 "MLD203CLN" H 5850 4324 50  0000 C CNN
+F 2 "" H 5850 3700 50  0001 C CNN
+F 3 "" H 5850 3700 50  0001 C CNN
+	1    5850 3700
+	1    0    0    -1
+$EndComp
+Wire Wire Line
+	6400 4150 6750 4150
+Wire Wire Line
+	6750 4150 6750 4200
+Wire Wire Line
+	6750 4200 6950 4200
+Wire Wire Line
+	6400 3700 6950 3700
+$Comp
+L Device:R_US R?
+U 1 1 5F1E131A
+P 6650 3850
+F 0 "R?" V 6445 3850 50  0000 C CNN
+F 1 "1k" V 6536 3850 50  0000 C CNN
+F 2 "" V 6690 3840 50  0001 C CNN
+F 3 "~" H 6650 3850 50  0001 C CNN
+	1    6650 3850
+	0    1    1    0
+$EndComp
+Wire Wire Line
+	6400 3850 6500 3850
+Wire Wire Line
+	6800 3850 6800 4000
+Wire Wire Line
+	6800 4000 6400 4000
+Text Label 6450 4000 0    50   ~ 0
+LD_CURR
 $EndSCHEMATC
